Commit message: add dxl_armed_turtlebot_gazebo.launch

File: dxl_armed_turtlebot/urdf/dynamixel_7dof_arm.urdf.xacro (robot description, xacro)
@@ -65,4 +65,21 @@
     </link>
   </macro>
+  <xacro:macro name="gazebo_arm_link" params="name color">
+    <gazebo reference="${name}">
+      <material>Gazebo/${color}</material>
+    </gazebo>
+  </xacro:macro>
+  <xacro:macro name="simple_transmission" params="name interface" >
+    <transmission name="${name}_trans">
+      <type>transmission_interface/SimpleTransmission</type>
+      <joint name="${name}">
+        <hardwareInterface>${interface}</hardwareInterface>
+      </joint>
+      <actuator name="${name}_motor">
+        <mechanicalReduction>10</mechanicalReduction>
+        <hardwareInterface>${interface}</hardwareInterface>
+      </actuator>
+    </transmission>
+  </xacro:macro>
   <xacro:macro name="dynamixel_7dof_arm" >
     <material name="black">
@@ -127,4 +144,35 @@
       <origin xyz="0.0 0.0 0.0" rpy="${M_PI/2} 0 ${M_PI/2}" />
     </xacro:ax12_hinge_revolute>
+    <!-- ros_control plugin -->
+    <gazebo>
+      <plugin name="gazebo_ros_control" filename="libgazebo_ros_control.so">
+        <robotNamespace>/dxl_armed_turtlebot</robotNamespace>
+      </plugin>
+      <plugin name="ground_truth" filename="libgazebo_ros_p3d.so">
+        <frameName>map</frameName>
+        <bodyName>base_footprint</bodyName>
+        <topicName>base_pose_ground_truth</topicName>
+        <updateRate>30.0</updateRate>
+      </plugin>
+    </gazebo>
+    <xacro:gazebo_arm_link name="arm_base_link" color="Black" />
+    <xacro:gazebo_arm_link name="arm_link0_link" color="Black" />
+    <xacro:gazebo_arm_link name="arm_link1_link" color="Gray" />
+    <xacro:gazebo_arm_link name="arm_link2_link" color="Black" />
+    <xacro:gazebo_arm_link name="arm_link2_motor_link" color="Black" />
+    <xacro:gazebo_arm_link name="arm_link3_link" color="Gray" />
+    <xacro:gazebo_arm_link name="arm_link3_motor_link" color="Black" />
+    <xacro:gazebo_arm_link name="arm_link4_link" color="Gray" />
+    <xacro:gazebo_arm_link name="arm_link5_link" color="Black" />
+    <xacro:gazebo_arm_link name="arm_link6_link" color="Black" />
+    <xacro:gazebo_arm_link name="arm_link6_motor_link" color="Black" />
+    <xacro:gazebo_arm_link name="arm_link7_link" color="Gray" />
+    <xacro:simple_transmission name="arm_link1_joint" interface="EffortJointInterface" />
+    <xacro:simple_transmission name="arm_link2_joint" interface="EffortJointInterface" />
+    <xacro:simple_transmission name="arm_link3_joint" interface="EffortJointInterface" />
+    <xacro:simple_transmission name="arm_link4_joint" interface="EffortJointInterface" />
+    <xacro:simple_transmission name="arm_link5_joint" interface="EffortJointInterface" />
+    <xacro:simple_transmission name="arm_link6_joint" interface="EffortJointInterface" />
+    <xacro:simple_transmission name="arm_link7_joint" interface="EffortJointInterface" />
   </xacro:macro>
 </robot>

Commit message: 7dof arm finished. moveit applied

File: dxl_armed_turtlebot/urdf/dynamixel_7dof_arm.urdf.xacro (robot description, xacro)
@@ -3,4 +3,33 @@
   <xacro:include filename="$(find dynamixel_urdf)/urdf/ax12.xacro" />
   <property name="M_PI" value="3.1415926535897931" />
+  <macro name="gripper_fixed" params="parent name color *origin">
+    <joint name="${name}_joint" type="fixed">
+      <insert_block name="origin" />
+      <parent link="${parent}"/>
+      <child link="${name}_link" />
+    </joint>
+    <link name="${name}_link">
+      <inertial>
+        <mass value="0.00001" />
+        <origin xyz="0 0 0" />
+        <inertia ixx="1.0" ixy="0.0" ixz="0.0"
+          iyy="1.0" iyz="0.0"
+          izz="1.0" />
+      </inertial>
+    <visual>
+      <origin xyz="0.04 0 0" rpy="0 0 0" />
+      <geometry>
+        <box size="0.08 0.01 0.030" />
+      </geometry>
+      <material name="white" />
+    </visual>
+      <collision>
+        <origin xyz="0.04 0.0 0.0" rpy="0 0 0" />
+        <geometry>
+          <box size="0.08 0.01 0.03"/>
+        </geometry>
+      </collision>
+    </link>
+  </macro>
   <macro name="dynamixel_ax12_joint" params="parent name color llimit ulimit vlimit *origin" >
     <joint name="${name}_joint" type="revolute">
@@ -65,4 +94,35 @@
     </link>
   </macro>
+ <!-- <macro name="ax12_hinge_revolute_axis_F3" params="parent name color llimit ulimit vlimit *origin *axis">
+    <joint name="${name}_joint" type="revolute">
+      <insert_block name="origin" />
+      <insert_block name="axis" />
+      <limit effort="30" velocity="${vlimit}" lower="${llimit}" upper="${ulimit}" />
+      <parent link="${parent}"/>
+      <child link="${name}_link" />
+    </joint>
+    <link name="${name}_link">
+      <inertial>
+        <mass value="0.00001" />
+        <origin xyz="0 0 0" />
+        <inertia ixx="1.0" ixy="0.0" ixz="0.0"
+          iyy="1.0" iyz="0.0"
+          izz="1.0" />
+      </inertial>
+      <visual>
+        <origin xyz=" 0 0 0 " rpy="0 0 0" />
+        <geometry>
+          <mesh filename="package://dynamixel_urdf/meshes/F3.stl" scale="0.001 0.001 0.001"/>
+        </geometry>
+        <material name="${color}"/>
+      </visual>
+      <collision>
+        <origin xyz="0.0 0.0 0.00775" rpy="0 0 0" />
+        <geometry>
+          <box size="0.025 0.0485 0.0375"/>
+        </geometry>
+      </collision>
+    </link>
+  </macro>-->
   <xacro:macro name="gazebo_arm_link" params="name color">
     <gazebo reference="${name}">
@@ -111,11 +171,19 @@
       <origin xyz="0.0 0.0 0.05" rpy="0 0 -${M_PI/2}" />
     </xacro:dynamixel_ax12_joint>
-    <xacro:dynamixel_ax12_tilt parent="arm_link2_link" name="arm_link2_motor" color="black">
-      <origin xyz="-0.06 0.0 0.02" rpy="0 0 0" />
+    <xacro:ax12_side_fixed parent="arm_link2_link" name="arm_link2_F31" color="white">
+      <origin xyz=" -0.039 0 0" rpy="${M_PI/2} 0 -${M_PI/2}" />
+    </xacro:ax12_side_fixed>
+    <xacro:ax12_side_fixed parent="arm_link2_F31_link" name="arm_link2_F32" color="white">
+      <origin xyz=" 0.0 0 0.0" rpy="${M_PI} 0 ${M_PI/2}" />
+    </xacro:ax12_side_fixed>
+<!-- -->
+    <xacro:dynamixel_ax12_tilt parent="arm_link2_F32_link" name="arm_link2_motor" color="white">
+      <origin xyz="0.025 0.0 -0.018" rpy="0 ${M_PI/2} 0" />
     </xacro:dynamixel_ax12_tilt>
+<!-- -->
     <xacro:ax12_hinge_revolute parent="arm_link2_motor_link" name="arm_link3"
                                llimit="-2.61" ulimit="2.61" vlimit="6.0"
                                color="white" >
-      <origin xyz="0.0 0.0 0.0" rpy="0 0 0" />
+      <origin xyz="0.0 0.0 0.0" rpy="0 0 ${M_PI}" />
     </xacro:ax12_hinge_revolute>
     <xacro:dynamixel_ax12_pan parent="arm_link3_link" name="arm_link3_motor" color="black">
@@ -132,10 +200,16 @@
       <origin xyz="0.0 0.0 0.0" rpy="0 -${M_PI/2} ${M_PI/2}" />
     </xacro:dynamixel_ax12_joint>
-    <xacro:dynamixel_ax12_joint parent="arm_link5_link" name="arm_link6"
+    <xacro:ax12_side_fixed parent="arm_link5_link" name="arm_link5_F3" color="white">
+      <origin xyz="-0.041 0 0.0" rpy="${M_PI/2} 0 -${M_PI/2}" />
+    </xacro:ax12_side_fixed>
+    <xacro:dynamixel_ax12_joint parent="arm_link5_F3_link" name="arm_link6"
                                llimit="-2.61" ulimit="2.61" vlimit="6.0" color="black">
-      <origin xyz="-0.07 0.0 0.0" rpy="-${M_PI/2} ${M_PI} -${M_PI/2}" />
+      <origin xyz="-0.0 0.0 0.023" rpy="-0 ${M_PI} 0" />
     </xacro:dynamixel_ax12_joint>
-    <xacro:dynamixel_ax12_pan parent="arm_link6_link" name="arm_link6_motor" color="black">
-      <origin xyz="0.0 0.03 -0.05" rpy="${M_PI/2} 0 ${M_PI/2}" />
+    <xacro:ax12_side_fixed parent="arm_link6_link" name="arm_link6_F3" color="white">
+      <origin xyz="-0.012 0 -0.025" rpy="-${M_PI} ${M_PI} ${M_PI/2}" />
+    </xacro:ax12_side_fixed>
+    <xacro:dynamixel_ax12_pan parent="arm_link6_F3_link" name="arm_link6_motor" color="black">
+      <origin xyz="-0.017 0.0 -0.024" rpy="${M_PI/2} 0 ${M_PI}" />
     </xacro:dynamixel_ax12_pan>
     <xacro:ax12_hinge_revolute parent="arm_link6_motor_link" name="arm_link7"
@@ -144,4 +218,20 @@
       <origin xyz="0.0 0.0 0.0" rpy="${M_PI/2} 0 ${M_PI/2}" />
     </xacro:ax12_hinge_revolute>
+    <xacro:gripper_fixed parent="arm_link7_link" name="gripper" color="white">
+      <origin xyz="-0.06 0.0 0.032" rpy="${M_PI/2} 0 0" />
+    </xacro:gripper_fixed>
+    <xacro:ax12_side_fixed parent="arm_link6_motor_link" name="gripper_F3" color="white">
+      <origin xyz="-0.037 0 0" rpy="${M_PI/2} ${M_PI} ${M_PI/2}" />
+    </xacro:ax12_side_fixed>
+    <xacro:gripper_fixed parent="gripper_F3_link" name="gripper_after_F3" color="white">
+      <origin xyz="0 0.0 -0.02" rpy="${M_PI/2} 0 0" />
+    </xacro:gripper_fixed>
+<!--
+    <xacro:gripper parent="arm_link7_link" name="gripper_link"
+                               llimit="-2.61" ulimit="2.61" vlimit="6.0"
+                               color="white" >
+      <origin xyz="0.0 0.0 0.0" rpy="${M_PI/2} 0 ${M_PI/2}" />
+    </xacro:gripper>
+-->
     <!-- ros_control plugin -->
     <gazebo>
@@ -156,9 +246,28 @@
       </plugin>
     </gazebo>
-    <xacro:gazebo_arm_link name="arm_base_link" color="Black" />
+    <xacro:gazebo_arm_link name="arm_base_link" color="Red" />
+    <xacro:gazebo_arm_link name="arm_link0_link" color="Orange" />
+    <xacro:gazebo_arm_link name="arm_link1_link" color="Yellow" />
+    <xacro:gazebo_arm_link name="arm_link2_link" color="Green" />
+    <xacro:gazebo_arm_link name="arm_link2_F31_link" color="Blue" />
+    <xacro:gazebo_arm_link name="arm_link2_F32_link" color="Purple" />
+    <xacro:gazebo_arm_link name="arm_link2_motor_link" color="Red" />
+    <xacro:gazebo_arm_link name="arm_link3_link" color="Orange" />
+    <xacro:gazebo_arm_link name="arm_link3_motor_link" color="Yellow" />
+    <xacro:gazebo_arm_link name="arm_link4_link" color="Green" />
+    <xacro:gazebo_arm_link name="arm_link5_link" color="Blue" />
+    <xacro:gazebo_arm_link name="arm_link5_F3_link" color="Purple" />
+    <xacro:gazebo_arm_link name="arm_link6_link" color="Red" />
+    <xacro:gazebo_arm_link name="arm_link6_F3_link" color="Orange" />
+    <xacro:gazebo_arm_link name="arm_link6_motor_link" color="Yellow" />
+    <xacro:gazebo_arm_link name="arm_link7_link" color="Green" />
+    <xacro:gazebo_arm_link name="gripper_link" color="Blue" />
+    <xacro:gazebo_arm_link name="gripper_after_F3_link" color="Purple" />
+    <xacro:gazebo_arm_link name="gripper_F3_link" color="Red" />
+<!--    <xacro:gazebo_arm_link name="arm_base_link" color="Black" />
     <xacro:gazebo_arm_link name="arm_link0_link" color="Black" />
     <xacro:gazebo_arm_link name="arm_link1_link" color="Gray" />
     <xacro:gazebo_arm_link name="arm_link2_link" color="Black" />
-    <xacro:gazebo_arm_link name="arm_link2_motor_link" color="Black" />
+    <xacro:gazebo_arm_link name="arm_link2_motor_link" color="Yellow" />
     <xacro:gazebo_arm_link name="arm_link3_link" color="Gray" />
     <xacro:gazebo_arm_link name="arm_link3_motor_link" color="Black" />
@@ -168,4 +277,6 @@
     <xacro:gazebo_arm_link name="arm_link6_motor_link" color="Black" />
     <xacro:gazebo_arm_link name="arm_link7_link" color="Gray" />
+-->
+    <xacro:gazebo_arm_link name="gripper_link_link" color="Gray" />
     <xacro:simple_transmission name="arm_link1_joint" interface="EffortJointInterface" />
     <xacro:simple_transmission name="arm_link2_joint" interface="EffortJointInterface" />

Commit message: dxl_armed_turtlebot/urdf/dynamixel_7dof_arm.urdf.xacro: correct urdf model for real robot

File: dxl_armed_turtlebot/urdf/dynamixel_7dof_arm.urdf.xacro (robot description, xacro)
@@ -3,4 +3,33 @@
   <xacro:include filename="$(find dynamixel_urdf)/urdf/ax12.xacro" />
   <property name="M_PI" value="3.1415926535897931" />
+  <macro name="gripper_fixed" params="parent name color *origin">
+    <joint name="${name}_joint" type="fixed">
+      <insert_block name="origin" />
+      <parent link="${parent}"/>
+      <child link="${name}_link" />
+    </joint>
+    <link name="${name}_link">
+      <inertial>
+        <mass value="0.00001" />
+        <origin xyz="0 0 0" />
+        <inertia ixx="1.0" ixy="0.0" ixz="0.0"
+          iyy="1.0" iyz="0.0"
+          izz="1.0" />
+      </inertial>
+      <visual>
+	<origin xyz="0.04 0 0" rpy="0 0 0" />
+	<geometry>
+          <box size="0.08 0.01 0.030" />
+	</geometry>
+	<material name="white" />
+      </visual>
+      <collision>
+        <origin xyz="0.04 0.0 0.0" rpy="0 0 0" />
+        <geometry>
+          <box size="0.08 0.01 0.03"/>
+        </geometry>
+      </collision>
+    </link>
+  </macro>
   <macro name="dynamixel_ax12_joint" params="parent name color llimit ulimit vlimit *origin" >
     <joint name="${name}_joint" type="revolute">
@@ -111,11 +140,17 @@
       <origin xyz="0.0 0.0 0.05" rpy="0 0 -${M_PI/2}" />
     </xacro:dynamixel_ax12_joint>
-    <xacro:dynamixel_ax12_tilt parent="arm_link2_link" name="arm_link2_motor" color="black">
-      <origin xyz="-0.06 0.0 0.02" rpy="0 0 0" />
+    <xacro:ax12_side_fixed parent="arm_link2_link" name="arm_link2_F31" color="white">
+      <origin xyz=" -0.039 0 0" rpy="${M_PI/2} 0 -${M_PI/2}" />
+    </xacro:ax12_side_fixed>
+    <xacro:ax12_side_fixed parent="arm_link2_F31_link" name="arm_link2_F32" color="white">
+      <origin xyz=" 0.0 0 0.0" rpy="${M_PI} 0 ${M_PI/2}" />
+    </xacro:ax12_side_fixed>
+    <xacro:dynamixel_ax12_tilt parent="arm_link2_F32_link" name="arm_link2_motor" color="white">
+      <origin xyz="0.025 0.0 -0.018" rpy="0 ${M_PI/2} 0" />
     </xacro:dynamixel_ax12_tilt>
     <xacro:ax12_hinge_revolute parent="arm_link2_motor_link" name="arm_link3"
                                llimit="-2.61" ulimit="2.61" vlimit="6.0"
                                color="white" >
-      <origin xyz="0.0 0.0 0.0" rpy="0 0 0" />
+      <origin xyz="0.0 0.0 0.0" rpy="0 0 ${M_PI}" />
     </xacro:ax12_hinge_revolute>
     <xacro:dynamixel_ax12_pan parent="arm_link3_link" name="arm_link3_motor" color="black">
@@ -132,10 +167,16 @@
       <origin xyz="0.0 0.0 0.0" rpy="0 -${M_PI/2} ${M_PI/2}" />
     </xacro:dynamixel_ax12_joint>
-    <xacro:dynamixel_ax12_joint parent="arm_link5_link" name="arm_link6"
+    <xacro:ax12_side_fixed parent="arm_link5_link" name="arm_link5_F3" color="white">
+      <origin xyz="-0.041 0 0.0" rpy="${M_PI/2} 0 -${M_PI/2}" />
+    </xacro:ax12_side_fixed>
+    <xacro:dynamixel_ax12_joint parent="arm_link5_F3_link" name="arm_link6"
                                llimit="-2.61" ulimit="2.61" vlimit="6.0" color="black">
-      <origin xyz="-0.07 0.0 0.0" rpy="-${M_PI/2} ${M_PI} -${M_PI/2}" />
+      <origin xyz="-0.0 0.0 0.023" rpy="-0 ${M_PI} 0" />
     </xacro:dynamixel_ax12_joint>
-    <xacro:dynamixel_ax12_pan parent="arm_link6_link" name="arm_link6_motor" color="black">
-      <origin xyz="0.0 0.03 -0.05" rpy="${M_PI/2} 0 ${M_PI/2}" />
+    <xacro:ax12_side_fixed parent="arm_link6_link" name="arm_link6_F3" color="white">
+      <origin xyz="-0.012 0 -0.025" rpy="-${M_PI} ${M_PI} ${M_PI/2}" />
+    </xacro:ax12_side_fixed>
+    <xacro:dynamixel_ax12_pan parent="arm_link6_F3_link" name="arm_link6_motor" color="black">
+      <origin xyz="-0.017 0.0 -0.024" rpy="${M_PI/2} 0 ${M_PI}" />
     </xacro:dynamixel_ax12_pan>
     <xacro:ax12_hinge_revolute parent="arm_link6_motor_link" name="arm_link7"
@@ -144,4 +185,13 @@
       <origin xyz="0.0 0.0 0.0" rpy="${M_PI/2} 0 ${M_PI/2}" />
     </xacro:ax12_hinge_revolute>
+    <xacro:gripper_fixed parent="arm_link7_link" name="gripper" color="white">
+      <origin xyz="-0.06 0.0 0.032" rpy="${M_PI/2} 0 0" />
+    </xacro:gripper_fixed>
+    <xacro:ax12_side_fixed parent="arm_link6_motor_link" name="gripper_F3" color="white">
+      <origin xyz="-0.037 0 0" rpy="${M_PI/2} ${M_PI} ${M_PI/2}" />
+    </xacro:ax12_side_fixed>
+    <xacro:gripper_fixed parent="gripper_F3_link" name="gripper_after_F3" color="white">
+      <origin xyz="0 0.0 -0.02" rpy="${M_PI/2} 0 0" />
+    </xacro:gripper_fixed>
     <!-- ros_control plugin -->
     <gazebo>
@@ -156,16 +206,24 @@
       </plugin>
     </gazebo>
-    <xacro:gazebo_arm_link name="arm_base_link" color="Black" />
-    <xacro:gazebo_arm_link name="arm_link0_link" color="Black" />
-    <xacro:gazebo_arm_link name="arm_link1_link" color="Gray" />
-    <xacro:gazebo_arm_link name="arm_link2_link" color="Black" />
-    <xacro:gazebo_arm_link name="arm_link2_motor_link" color="Black" />
-    <xacro:gazebo_arm_link name="arm_link3_link" color="Gray" />
-    <xacro:gazebo_arm_link name="arm_link3_motor_link" color="Black" />
-    <xacro:gazebo_arm_link name="arm_link4_link" color="Gray" />
-    <xacro:gazebo_arm_link name="arm_link5_link" color="Black" />
-    <xacro:gazebo_arm_link name="arm_link6_link" color="Black" />
-    <xacro:gazebo_arm_link name="arm_link6_motor_link" color="Black" />
-    <xacro:gazebo_arm_link name="arm_link7_link" color="Gray" />
+    <xacro:gazebo_arm_link name="arm_base_link" color="Red" />
+    <xacro:gazebo_arm_link name="arm_link0_link" color="Orange" />
+    <xacro:gazebo_arm_link name="arm_link1_link" color="Yellow" />
+    <xacro:gazebo_arm_link name="arm_link2_link" color="Green" />
+    <xacro:gazebo_arm_link name="arm_link2_F31_link" color="Blue" />
+    <xacro:gazebo_arm_link name="arm_link2_F32_link" color="Purple" />
+    <xacro:gazebo_arm_link name="arm_link2_motor_link" color="Red" />
+    <xacro:gazebo_arm_link name="arm_link3_link" color="Orange" />
+    <xacro:gazebo_arm_link name="arm_link3_motor_link" color="Yellow" />
+    <xacro:gazebo_arm_link name="arm_link4_link" color="Green" />
+    <xacro:gazebo_arm_link name="arm_link5_link" color="Blue" />
+    <xacro:gazebo_arm_link name="arm_link5_F3_link" color="Purple" />
+    <xacro:gazebo_arm_link name="arm_link6_link" color="Red" />
+    <xacro:gazebo_arm_link name="arm_link6_F3_link" color="Orange" />
+    <xacro:gazebo_arm_link name="arm_link6_motor_link" color="Yellow" />
+    <xacro:gazebo_arm_link name="arm_link7_link" color="Green" />
+    <xacro:gazebo_arm_link name="gripper_link" color="Blue" />
+    <xacro:gazebo_arm_link name="gripper_after_F3_link" color="Purple" />
+    <xacro:gazebo_arm_link name="gripper_F3_link" color="Red" />
+    <xacro:gazebo_arm_link name="gripper_link_link" color="Gray" />
     <xacro:simple_transmission name="arm_link1_joint" interface="EffortJointInterface" />
     <xacro:simple_transmission name="arm_link2_joint" interface="EffortJointInterface" />
