Commit message: Add gripper model

File: dxl_armed_turtlebot/urdf/dynamixel_7dof_arm.urdf.xacro (robot description, xacro)
@@ -33,5 +33,5 @@
       <parent link="${parent}"/>
       <child link="${name}_link" />
-      <dynamics damping="0" />
+      <dynamics damping="0.1" />
     </joint>
     <link name="${name}_link">
@@ -128,4 +128,33 @@
         <geometry>
           <box size="0.025 0.0485 ${0.0375-0.03}"/>
+        </geometry>
+      </collision>
+    </link>
+  </macro>
+  <macro name="half_grpper" params="parent name color *origin">
+    <joint name="${name}_joint" type="fixed">
+      <insert_block name="origin" />
+      <parent link="${parent}"/>
+      <child link="${name}_link" />
+    </joint>
+    <link name="${name}_link">
+      <inertial>
+        <origin xyz=" 0.025 0 0.003" rpy="0 0 0" />
+        <mass value="0.013" />
+        <inertia ixx="0.0" ixy="0.0" ixz="0.0"
+                 iyy="0.00002" iyz="0.0"
+                 izz="0.00002" />
+      </inertial>
+      <visual>
+        <origin xyz=" 0 0 0 " rpy="0 0 0" />
+        <geometry>
+          <mesh filename="package://dynamixel_urdf/meshes/dxl_gripper.stl" scale="0.001 0.001 0.001"/>
+        </geometry>
+        <material name="${color}"/>
+      </visual>
+      <collision>
+        <origin xyz="0.027 0.0 0.01" rpy="0 0 0" />
+        <geometry>
+          <box size="0.08 0.04 0.02"/>
         </geometry>
       </collision>
@@ -220,4 +249,10 @@
       <axis xyz="0 1 0"/>
     </xacro:ax12_hinge_revolute_axis>
+    <xacro:half_grpper parent="arm_link7_link" name="arm_gripper_left" color="white" >
+      <origin xyz="0.0 0.0 0.027" rpy="0 0 ${M_PI}" />
+    </xacro:half_grpper>
+    <xacro:half_grpper parent="arm_link6_motor_link" name="arm_gripper_right" color="white" >
+      <origin xyz="-0.041 0.0 0.0" rpy="${M_PI/2} 0 ${-M_PI/2}" />
+    </xacro:half_grpper>
     <!-- ros_control plugin -->
     <gazebo>
@@ -242,4 +277,6 @@
     <xacro:gazebo_arm_link name="arm_link6_motor_link" color="Black" />
     <xacro:gazebo_arm_link name="arm_link7_link" color="Grey" />
+    <xacro:gazebo_arm_link name="arm_gripper_left" color="Grey" />
+    <xacro:gazebo_arm_link name="arm_gripper_right" color="Grey" />
     <xacro:simple_transmission name="arm_link1_joint" interface="${joint_interface}" />
     <xacro:simple_transmission name="arm_link2_joint" interface="${joint_interface}" />
