Commit message: Update the arm root position

File: dxl_armed_turtlebot/urdf/robot.urdf.xacro (robot description, xacro)
@@ -12,5 +12,5 @@
     <parent link="plate_top_link"/>
     <child link="arm_base_link"/>
-    <origin xyz="0.15 0 0.025" rpy="0 0 0" />
+    <origin xyz="0.122 0 -0.025" rpy="0 0 0" />
   </joint>
 </robot>

Commit message: Move arm urdf file under dynamxiel_7dof_arm

File: dxl_armed_turtlebot/urdf/robot.urdf.xacro (robot description, xacro)
@@ -4,5 +4,5 @@
   <xacro:include filename="$(find turtlebot_description)/urdf/stacks/hexagons.urdf.xacro" />
   <xacro:include filename="$(find turtlebot_description)/urdf/sensors/kinect.urdf.xacro" />
-  <xacro:include filename="$(find dxl_armed_turtlebot)/urdf/dynamixel_7dof_arm.urdf.xacro" />
+  <xacro:include filename="$(find dynamixel_7dof_arm)/urdf/dynamixel_7dof_arm.urdf.xacro" />
   <kobuki/>
   <stack_hexagons parent="base_link"/>

File: dynamixel_7dof_arm/urdf/dynamixel_7dof_arm.urdf.xacro (robot description, xacro)
@@ -42,5 +42,5 @@
         <origin xyz=" 0 0 0 " rpy="1.57 0 1.57" />
         <geometry>
-          <mesh filename="package://dynamixel_urdf/meshes/ax12.stl" scale="0.001 0.001 0.001"/>
+          <mesh filename="package://dynamixel_7dof_arm/urdf/meshes/ax12.stl" scale="0.001 0.001 0.001"/>
         </geometry>
         <material name="${color}"/>
@@ -67,5 +67,5 @@
         <origin xyz=" 0 0 0 " rpy="1.57 0 1.57" />
         <geometry>
-          <mesh filename="package://dynamixel_urdf/meshes/ax12.stl" scale="0.001 0.001 0.001"/>
+          <mesh filename="package://dynamixel_7dof_arm/urdf/meshes/ax12.stl" scale="0.001 0.001 0.001"/>
         </geometry>
         <material name="${color}"/>
@@ -92,5 +92,5 @@
         <origin xyz=" 0 0 0 " rpy="0 0 0" />
         <geometry>
-          <mesh filename="package://dynamixel_urdf/meshes/ax12.stl" scale="0.001 0.001 0.001"/>
+          <mesh filename="package://dynamixel_7dof_arm/urdf/meshes/ax12.stl" scale="0.001 0.001 0.001"/>
         </geometry>
         <material name="${color}"/>
@@ -120,5 +120,5 @@
         <origin xyz=" 0 0 0 " rpy="0 0 0" />
         <geometry>
-          <mesh filename="package://dynamixel_urdf/meshes/F2.stl" scale="0.001 0.001 0.001"/>
+          <mesh filename="package://dynamixel_7dof_arm/urdf/meshes/F2.stl" scale="0.001 0.001 0.001"/>
         </geometry>
         <material name="${color}"/>
@@ -149,5 +149,5 @@
         <origin xyz=" 0 0 0 " rpy="0 0 0" />
         <geometry>
-          <mesh filename="package://dynamixel_urdf/meshes/dxl_gripper.stl" scale="0.001 0.001 0.001"/>
+          <mesh filename="package://dynamixel_7dof_arm/urdf/meshes/dxl_gripper.stl" scale="0.001 0.001 0.001"/>
         </geometry>
         <material name="${color}"/>

Commit message: Update the length of arm base hinge

File: dxl_armed_turtlebot/urdf/robot.urdf.xacro (robot description, xacro)
@@ -12,5 +12,5 @@
     <parent link="plate_top_link"/>
     <child link="arm_base_link"/>
-    <origin xyz="0.122 0 -0.025" rpy="0 0 0" />
+    <origin xyz="0.182 0 -0.025" rpy="0 0 0" />
   </joint>
 </robot>

File: dynamixel_7dof_arm/urdf/dynamixel_7dof_arm.urdf.xacro (robot description, xacro)
@@ -193,7 +193,7 @@
     <link name="arm_base_link">
       <visual>
-        <origin xyz="-0.02 0.0 0.0" rpy="0 0 0" />
-        <geometry>
-          <box size="0.04 0.03 0.04" />
+        <origin xyz="-0.05 0.0 0.0" rpy="0 0 0" />
+        <geometry>
+          <box size="0.1 0.03 0.04" />
         </geometry>
         <material name="white" />
