Commit message: Change the joint name form "arm_link${num}_joint" to "arm_joint${num}", in order to match the naming rule in real robot and eus model

File: dynamixel_7dof_arm/urdf/dynamixel_7dof_arm.urdf.xacro (robot description, xacro)
@@ -25,6 +25,6 @@
     </inertial>
   </xacro:macro>
-  <macro name="dynamixel_ax12_joint" params="parent name color llimit ulimit vlimit *origin" >
-    <joint name="${name}_joint" type="revolute">
+  <macro name="dynamixel_ax12_joint" params="parent name joint_name color llimit ulimit vlimit *origin" >
+    <joint name="${joint_name}" type="revolute">
       <insert_block name="origin" />
       <axis xyz="0 0 1"/>
@@ -104,6 +104,6 @@
     </link>
   </macro>
-  <macro name="ax12_hinge_revolute_axis" params="parent name color llimit ulimit vlimit *origin *axis">
-    <joint name="${name}_joint" type="revolute">
+  <macro name="ax12_hinge_revolute_axis" params="parent name joint_name color llimit ulimit vlimit *origin *axis">
+    <joint name="${joint_name}" type="revolute">
       <insert_block name="origin" />
       <insert_block name="axis" />
@@ -203,5 +203,5 @@
       <origin xyz="0.045 0 0.0" rpy="${M_PI} 0 0" />
     </xacro:dynamixel_ax12_pan>
-    <xacro:ax12_hinge_revolute_axis parent="arm_link0_link" name="arm_link1"
+    <xacro:ax12_hinge_revolute_axis parent="arm_link0_link" name="arm_link1" joint_name="arm_joint1"
                                llimit="-2.0944" ulimit="2.0944" vlimit="${vlimit}"
                                color="white" >
@@ -209,5 +209,5 @@
       <axis xyz="0 1 0"/>
     </xacro:ax12_hinge_revolute_axis>
-    <xacro:dynamixel_ax12_joint parent="arm_link1_link" name="arm_link2"
+    <xacro:dynamixel_ax12_joint parent="arm_link1_link" name="arm_link2" joint_name="arm_joint2"
                                llimit="-2.61" ulimit="2.61" vlimit="${vlimit}"
                                color="black" >
@@ -217,5 +217,5 @@
       <origin xyz="-0.06 0.0 0.02" rpy="0 0 0" />
     </xacro:dynamixel_ax12_tilt>
-    <xacro:ax12_hinge_revolute_axis parent="arm_link2_motor_link" name="arm_link3"
+    <xacro:ax12_hinge_revolute_axis parent="arm_link2_motor_link" name="arm_link3" joint_name="arm_joint3"
                                llimit="-2.0944" ulimit="2.0944" vlimit="${vlimit}"
                                color="white" >
@@ -226,5 +226,5 @@
       <origin xyz="-0.01 0.0 0.055" rpy="${M_PI} ${M_PI} 0" />
     </xacro:dynamixel_ax12_pan>
-    <xacro:ax12_hinge_revolute_axis parent="arm_link3_motor_link" name="arm_link4"
+    <xacro:ax12_hinge_revolute_axis parent="arm_link3_motor_link" name="arm_link4" joint_name="arm_joint4"
                                llimit="-2.61" ulimit="2.61" vlimit="${vlimit}"
                                color="white" >
@@ -232,9 +232,9 @@
       <axis xyz="0 0 1" />
     </xacro:ax12_hinge_revolute_axis>
-    <xacro:dynamixel_ax12_joint parent="arm_link4_link" name="arm_link5"
+    <xacro:dynamixel_ax12_joint parent="arm_link4_link" name="arm_link5" joint_name="arm_joint5"
                                llimit="-2.0944" ulimit="1.5708" vlimit="${vlimit}" color="black">
       <origin xyz="0.0 0.0 0.0" rpy="0 -${M_PI/2} ${M_PI/2}" />
     </xacro:dynamixel_ax12_joint>
-    <xacro:dynamixel_ax12_joint parent="arm_link5_link" name="arm_link6"
+    <xacro:dynamixel_ax12_joint parent="arm_link5_link" name="arm_link6" joint_name="arm_joint6"
                                llimit="-2.61" ulimit="2.61" vlimit="${vlimit}" color="black">
       <origin xyz="-0.07 0.0 0.0" rpy="-${M_PI/2} ${M_PI} -${M_PI/2}" />
@@ -243,5 +243,5 @@
       <origin xyz="0.0 0.03 -0.05" rpy="${M_PI/2} 0 ${M_PI/2}" />
     </xacro:dynamixel_ax12_pan>
-    <xacro:ax12_hinge_revolute_axis parent="arm_link6_motor_link" name="arm_link7"
+    <xacro:ax12_hinge_revolute_axis parent="arm_link6_motor_link" name="arm_link7" joint_name="gripper_joint"
                                llimit="-1.5708" ulimit="1.5708" vlimit="${vlimit}"
                                color="white" >
@@ -287,11 +287,11 @@
       <mu2>0.8</mu2>
     </gazebo>
-    <xacro:simple_transmission name="arm_link1_joint" interface="${joint_interface}" />
-    <xacro:simple_transmission name="arm_link2_joint" interface="${joint_interface}" />
-    <xacro:simple_transmission name="arm_link3_joint" interface="${joint_interface}" />
-    <xacro:simple_transmission name="arm_link4_joint" interface="${joint_interface}" />
-    <xacro:simple_transmission name="arm_link5_joint" interface="${joint_interface}" />
-    <xacro:simple_transmission name="arm_link6_joint" interface="${joint_interface}" />
-    <xacro:simple_transmission name="arm_link7_joint" interface="${joint_interface}" />
+    <xacro:simple_transmission name="arm_joint1" interface="${joint_interface}" />
+    <xacro:simple_transmission name="arm_joint2" interface="${joint_interface}" />
+    <xacro:simple_transmission name="arm_joint3" interface="${joint_interface}" />
+    <xacro:simple_transmission name="arm_joint4" interface="${joint_interface}" />
+    <xacro:simple_transmission name="arm_joint5" interface="${joint_interface}" />
+    <xacro:simple_transmission name="arm_joint6" interface="${joint_interface}" />
+    <xacro:simple_transmission name="gripper_joint" interface="${joint_interface}" />
   </xacro:macro>
 </robot>

Commit message: Update the urdf model for dxynamixel 7dof arm to match the true robot model

File: dynamixel_7dof_arm/urdf/dynamixel_7dof_arm.urdf.xacro (robot description, xacro)
@@ -25,8 +25,8 @@
     </inertial>
   </xacro:macro>
-  <macro name="dynamixel_ax12_joint" params="parent name joint_name color llimit ulimit vlimit *origin" >
+  <macro name="dynamixel_ax12_joint" params="parent name joint_name color llimit ulimit vlimit *origin *axis" >
     <joint name="${joint_name}" type="revolute">
       <insert_block name="origin" />
-      <axis xyz="0 0 1"/>
+      <insert_block name="axis" />
       <limit effort="${elimit}" velocity="${vlimit}" lower="${llimit - 0.1}" upper="${ulimit + 0.1}" />
 <!--      <safety_controller soft_lower_limit="${llimit}" soft_upper_limit="${ulimit}" k_position="1" k_velocity="1" /> -->
@@ -201,5 +201,5 @@
     </link>
     <xacro:dynamixel_ax12_pan parent="arm_base_link" name="arm_link0" color="black">
-      <origin xyz="0.045 0 0.0" rpy="${M_PI} 0 0" />
+      <origin xyz="0.045 0 0.0" rpy="0 0 0" />
     </xacro:dynamixel_ax12_pan>
     <xacro:ax12_hinge_revolute_axis parent="arm_link0_link" name="arm_link1" joint_name="arm_joint1"
@@ -212,8 +212,9 @@
                                llimit="-2.61" ulimit="2.61" vlimit="${vlimit}"
                                color="black" >
-      <origin xyz="0.0 0.0 0.05" rpy="0 0 -${M_PI/2}" />
+      <origin xyz="0.0 0.0 0.05" rpy="${M_PI} 0 ${M_PI/2}" />
+      <axis xyz="0 0 -1" />
     </xacro:dynamixel_ax12_joint>
     <xacro:dynamixel_ax12_tilt parent="arm_link2_link" name="arm_link2_motor" color="black">
-      <origin xyz="-0.06 0.0 0.02" rpy="0 0 0" />
+      <origin xyz="-0.06 0.0 -0.02" rpy="${M_PI} 0 0" />
     </xacro:dynamixel_ax12_tilt>
     <xacro:ax12_hinge_revolute_axis parent="arm_link2_motor_link" name="arm_link3" joint_name="arm_joint3"
@@ -224,5 +225,5 @@
     </xacro:ax12_hinge_revolute_axis>
     <xacro:dynamixel_ax12_pan parent="arm_link3_link" name="arm_link3_motor" color="black">
-      <origin xyz="-0.01 0.0 0.055" rpy="${M_PI} ${M_PI} 0" />
+      <origin xyz="-0.014 0.0 0.055" rpy="${M_PI} ${M_PI} 0" />
     </xacro:dynamixel_ax12_pan>
     <xacro:ax12_hinge_revolute_axis parent="arm_link3_motor_link" name="arm_link4" joint_name="arm_joint4"
@@ -230,13 +231,15 @@
                                color="white" >
       <origin xyz="0.0 0.0 0.05" rpy="0 ${M_PI} 0" />
-      <axis xyz="0 0 1" />
+      <axis xyz="0 0 -1" />
     </xacro:ax12_hinge_revolute_axis>
     <xacro:dynamixel_ax12_joint parent="arm_link4_link" name="arm_link5" joint_name="arm_joint5"
                                llimit="-2.0944" ulimit="1.5708" vlimit="${vlimit}" color="black">
       <origin xyz="0.0 0.0 0.0" rpy="0 -${M_PI/2} ${M_PI/2}" />
+      <axis xyz="0 0 1" />
     </xacro:dynamixel_ax12_joint>
     <xacro:dynamixel_ax12_joint parent="arm_link5_link" name="arm_link6" joint_name="arm_joint6"
                                llimit="-2.61" ulimit="2.61" vlimit="${vlimit}" color="black">
       <origin xyz="-0.07 0.0 0.0" rpy="-${M_PI/2} ${M_PI} -${M_PI/2}" />
+      <axis xyz="0 0 -1" />
     </xacro:dynamixel_ax12_joint>
     <xacro:dynamixel_ax12_pan parent="arm_link6_link" name="arm_link6_motor" color="black">

Commit message: update deprecated urdf/xacro tags

File: dynamixel_7dof_arm/urdf/dynamixel_7dof_arm.urdf.xacro (robot description, xacro)
@@ -2,9 +2,9 @@
 <robot xmlns:xacro="http://ros.org/wiki/xacro" >
   <!-- <xacro:include filename="$(find dynamixel_urdf)/urdf/ax12.xacro" /> -->
-  <property name="M_PI" value="3.1415926535897931" />
-  <property name="elimit" value="1.5" />
-  <property name="vlimit" value="6.0" />
-  <!-- <property name="joint_interface" value="EffortJointInterface" /> -->
-  <property name="joint_interface" value="VelocityJointInterface" />
+  <xacro:property name="M_PI" value="3.1415926535897931" />
+  <xacro:property name="elimit" value="1.5" />
+  <xacro:property name="vlimit" value="6.0" />
+  <!-- <xacro:property name="joint_interface" value="EffortJointInterface" /> -->
+  <xacro:property name="joint_interface" value="VelocityJointInterface" />
   <!-- Macro for the inertia of a box -->
   <xacro:macro name="box_inertia" params="x y z mass">
@@ -25,7 +25,7 @@
     </inertial>
   </xacro:macro>
-  <macro name="dynamixel_ax12_joint" params="parent name color llimit ulimit vlimit *origin" >
+  <xacro:macro name="dynamixel_ax12_joint" params="parent name color llimit ulimit vlimit *origin" >
     <joint name="${name}_joint" type="revolute">
-      <insert_block name="origin" />
+      <xacro:insert_block name="origin" />
       <axis xyz="0 0 1"/>
       <limit effort="${elimit}" velocity="${vlimit}" lower="${llimit - 0.1}" upper="${ulimit + 0.1}" />
@@ -53,8 +53,8 @@
       </collision>
     </link>
-  </macro>
-  <macro name="dynamixel_ax12_pan" params="parent name color *origin" >
+  </xacro:macro>
+  <xacro:macro name="dynamixel_ax12_pan" params="parent name color *origin" >
     <joint name="${name}_joint" type="fixed">
-      <insert_block name="origin" />
+      <xacro:insert_block name="origin" />
       <parent link="${parent}"/>
       <child link="${name}_link" />
@@ -78,8 +78,8 @@
       </collision>
     </link>
-  </macro>
-  <macro name="dynamixel_ax12_tilt" params="parent name color *origin" >
+  </xacro:macro>
+  <xacro:macro name="dynamixel_ax12_tilt" params="parent name color *origin" >
     <joint name="${name}_joint" type="fixed">
-      <insert_block name="origin" />
+      <xacro:insert_block name="origin" />
       <parent link="${parent}"/>
       <child link="${name}_link" />
@@ -103,9 +103,9 @@
       </collision>
     </link>
-  </macro>
-  <macro name="ax12_hinge_revolute_axis" params="parent name color llimit ulimit vlimit *origin *axis">
+  </xacro:macro>
+  <xacro:macro name="ax12_hinge_revolute_axis" params="parent name color llimit ulimit vlimit *origin *axis">
     <joint name="${name}_joint" type="revolute">
-      <insert_block name="origin" />
-      <insert_block name="axis" />
+      <xacro:insert_block name="origin" />
+      <xacro:insert_block name="axis" />
       <limit effort="${elimit}" velocity="${vlimit}" lower="${llimit - 0.1}" upper="${ulimit + 0.1}" />
       <safety_controller soft_lower_limit="${llimit}" soft_upper_limit="${ulimit}" k_position="1" k_velocity="1" />
@@ -131,8 +131,8 @@
       </collision>
     </link>
-  </macro>
-  <macro name="half_grpper" params="parent name color *origin">
+  </xacro:macro>
+  <xacro:macro name="half_grpper" params="parent name color *origin">
     <joint name="${name}_joint" type="fixed">
-      <insert_block name="origin" />
+      <xacro:insert_block name="origin" />
       <parent link="${parent}"/>
       <child link="${name}_link" />
@@ -160,5 +160,5 @@
       </collision>
     </link>
-  </macro>
+  </xacro:macro>
   <xacro:macro name="gazebo_arm_link" params="name color">
     <gazebo reference="${name}">

Commit message: fix xacro : property -> xacro:property

File: dynamixel_7dof_arm/urdf/dynamixel_7dof_arm.urdf.xacro (robot description, xacro)
@@ -2,10 +2,10 @@
 <robot xmlns:xacro="http://ros.org/wiki/xacro" >
   <!-- <xacro:include filename="$(find dynamixel_urdf)/urdf/ax12.xacro" /> -->
-  <property name="M_PI" value="3.1415926535897931" />
-  <property name="elimit" value="1.5" />
-  <property name="vlimit" value="6.0" />
+  <xacro:property name="M_PI" value="3.1415926535897931" />
+  <xacro:property name="elimit" value="1.5" />
+  <xacro:property name="vlimit" value="6.0" />
   <!-- <property name="joint_interface" value="EffortJointInterface" /> -->
-  <property name="joint_interface" value="VelocityJointInterface" />
-  <property name="joint_interface" value="hardware_interface/VelocityJointInterface" />
+  <xacro:property name="joint_interface" value="VelocityJointInterface" />
+  <xacro:property name="joint_interface" value="hardware_interface/VelocityJointInterface" />
   <!-- Macro for the inertia of a box -->
   <xacro:macro name="box_inertia" params="x y z mass">

Commit message: fix xacro: deprecated: xacro tags should be prepended with 'xacro' xml namespace. Use the following script to fix incorrect usage:         find . -iname *.xacro | xargs sed -i 's#<\([/]\?\)\(if\|unless\|include\|arg\|property\|macro\|insert_block\)#<\1xacro:\2#g' when processing file: /home/k-okada/catkin_ws/ws_enshu/src/robot-programming/dynamixel_7dof_arm/urdf/dynamixel_7dof_arm.urdf.xacro

File: dynamixel_7dof_arm/urdf/dynamixel_7dof_arm.urdf.xacro (robot description, xacro)
@@ -5,5 +5,5 @@
   <xacro:property name="elimit" value="1.5" />
   <xacro:property name="vlimit" value="6.0" />
-  <!-- <property name="joint_interface" value="EffortJointInterface" /> -->
+  <!-- <xacro:property name="joint_interface" value="EffortJointInterface" /> -->
   <xacro:property name="joint_interface" value="VelocityJointInterface" />
   <xacro:property name="joint_interface" value="hardware_interface/VelocityJointInterface" />
@@ -26,8 +26,8 @@
     </inertial>
   </xacro:macro>
-  <macro name="dynamixel_ax12_joint" params="parent name joint_name color llimit ulimit vlimit *origin *axis" >
+  <xacro:macro name="dynamixel_ax12_joint" params="parent name joint_name color llimit ulimit vlimit *origin *axis" >
     <joint name="${joint_name}" type="revolute">
-      <insert_block name="origin" />
-      <insert_block name="axis" />
+      <xacro:insert_block name="origin" />
+      <xacro:insert_block name="axis" />
       <limit effort="${elimit}" velocity="${vlimit}" lower="${llimit - 0.1}" upper="${ulimit + 0.1}" />
 <!--      <safety_controller soft_lower_limit="${llimit}" soft_upper_limit="${ulimit}" k_position="1" k_velocity="1" /> -->
@@ -54,8 +54,8 @@
       </collision>
     </link>
-  </macro>
-  <macro name="dynamixel_ax12_pan" params="parent name color *origin" >
+  </xacro:macro>
+  <xacro:macro name="dynamixel_ax12_pan" params="parent name color *origin" >
     <joint name="${name}_joint" type="fixed">
-      <insert_block name="origin" />
+      <xacro:insert_block name="origin" />
       <parent link="${parent}"/>
       <child link="${name}_link" />
@@ -79,8 +79,8 @@
       </collision>
     </link>
-  </macro>
-  <macro name="dynamixel_ax12_tilt" params="parent name color *origin" >
+  </xacro:macro>
+  <xacro:macro name="dynamixel_ax12_tilt" params="parent name color *origin" >
     <joint name="${name}_joint" type="fixed">
-      <insert_block name="origin" />
+      <xacro:insert_block name="origin" />
       <parent link="${parent}"/>
       <child link="${name}_link" />
@@ -104,9 +104,9 @@
       </collision>
     </link>
-  </macro>
-  <macro name="ax12_hinge_revolute_axis" params="parent name joint_name color llimit ulimit vlimit *origin *axis">
+  </xacro:macro>
+  <xacro:macro name="ax12_hinge_revolute_axis" params="parent name joint_name color llimit ulimit vlimit *origin *axis">
     <joint name="${joint_name}" type="revolute">
-      <insert_block name="origin" />
-      <insert_block name="axis" />
+      <xacro:insert_block name="origin" />
+      <xacro:insert_block name="axis" />
       <limit effort="${elimit}" velocity="${vlimit}" lower="${llimit - 0.1}" upper="${ulimit + 0.1}" />
 <!--      <safety_controller soft_lower_limit="${llimit}" soft_upper_limit="${ulimit}" k_position="1" k_velocity="1" /> -->
@@ -132,8 +132,8 @@
       </collision>
     </link>
-  </macro>
-  <macro name="half_grpper" params="parent name color *origin">
+  </xacro:macro>
+  <xacro:macro name="half_grpper" params="parent name color *origin">
     <joint name="${name}_joint" type="fixed">
-      <insert_block name="origin" />
+      <xacro:insert_block name="origin" />
       <parent link="${parent}"/>
       <child link="${name}_link" />
@@ -161,5 +161,5 @@
       </collision>
     </link>
-  </macro>
+  </xacro:macro>
   <xacro:macro name="gazebo_arm_link" params="name color">
     <gazebo reference="${name}">
