Commit message: update robot model

File: mechatrobot/urdf/robot.urdf (robot description, URDF)
Before this commit: robot robot, 4 links, 3 joints
Links:
- removed link joint_link
- removed link range
- added link link1; visual box size=0.01 0.1 0.005
- added link range_sensor; visual mesh filename=package://mechatrobot/urdf/HC-SR04.STL scale=0.001 0.001 0.001
- link base_link: geometry visual box size=0.053 0.082 0.01
- link motor_link: geometry visual mesh filename=package://mechatrobot/urdf/28BYJ-48.STL scale=0.001 0.001 0.001
Joints:
- removed joint base_to_range
- added joint base_to_sensor: type fixed, parent base_link, child range_sensor, origin xyz=0.02 -0.03 0.02
- joint base_to_motor: origin xyz=-0.04 0 0 -> xyz=0 0.08 0 rpy=0 0 0
- joint joint1: axis 0 0 1 -> 0 0 -1; child joint_link -> link1; origin xyz=0 0 0.1 -> xyz=-0.008 0 0.03
