Commit message: [kx-pr2] Use base laser scan

File: kx_pr2/kx_pr2_bringup/urdf/kx_pr2.urdf (robot description, URDF)
Before this commit: robot kx_pr2, 10 links, 9 joints
Links:
- added link base_laser, mass 0.1; collision cylinder length=0.01 radius=0.05; visual cylinder length=0.01 radius=0.05
Joints:
- added joint base_laser_joint: type fixed, parent base_link, child base_laser, origin xyz=0.1 0 -0.0 rpy=0 0 0

Commit message: [kx-pr2] Fixed wheel parameteres

File: kx_pr2/kx_pr2_bringup/urdf/kx_pr2.urdf (robot description, URDF)
Before this commit: robot kx_pr2, 11 links, 10 joints
Links:
- link base_laser: mass 0.1 -> None; geometry 
