Commit message: [jedy_description] Fixed coordinates

File: jedy/jedy_description/urdf/jedy.urdf (robot description, URDF)
Before this commit: robot jedy, 25 links, 24 joints
Links:
- added link real_base_link, mass 0.642084743261537; collision mesh filename=package://jedy_description/meshes/base_link.dae; visual mesh filename=package://jedy_description/meshes/base_link.dae
- link base_link: mass 0.642084743261537 -> None; geometry 
Joints:
- added joint pseudo_base_joint: type fixed, parent base_link, child real_base_link, origin xyz=0 0 0 rpy=1.5707926535897931 0 1.5707926535897931, axis 0. 0. 0., limit lower=0 upper=0 effort=0 velocity=0
- joint front_left_wheel_joint: parent base_link -> real_base_link
- joint front_right_wheel_joint: parent base_link -> real_base_link
- joint head_joint0: parent base_link -> real_base_link
- joint larm_joint0: parent base_link -> real_base_link
- joint rarm_joint0: parent base_link -> real_base_link
- joint rear_left_wheel_joint: parent base_link -> real_base_link
- joint rear_right_wheel_joint: parent base_link -> real_base_link

Commit message: [jedy_description] Fixed joint limit

File: jedy/jedy_description/urdf/jedy.urdf (robot description, URDF)
Before this commit: robot jedy, 26 links, 25 joints
Joints:
- joint larm_joint3: limit lower=0.0 upper=-2.35 effort=0.48 velocity=6.55 -> lower=-2.35 upper=2.35 effort=0.48 velocity=6.55
- joint rarm_joint3: limit lower=0.0 upper=-2.35 effort=0.48 velocity=6.55 -> lower=-2.35 upper=2.35 effort=0.48 velocity=6.55

Commit message: [jedy_description] Use cylinder

File: jedy/jedy_description/urdf/jedy.urdf (robot description, URDF)
Before this commit: robot jedy, 26 links, 25 joints
Links:
- link front_left_wheel_link: geometry collision cylinder length=0.02 radius=0.03; visual mesh filename=package://jedy_description/meshes/front_left_wheel_link.dae
- link front_right_wheel_link: geometry collision cylinder length=0.02 radius=0.03; visual mesh filename=package://jedy_description/meshes/front_right_wheel_link.dae
- link rear_left_wheel_link: geometry collision cylinder length=0.02 radius=0.03; visual mesh filename=package://jedy_description/meshes/rear_left_wheel_link.dae
- link rear_right_wheel_link: geometry collision cylinder length=0.02 radius=0.03; visual mesh filename=package://jedy_description/meshes/rear_right_wheel_link.dae

Commit message: Modified parameters for gazebo

File: jedy/jedy_description/urdf/jedy.urdf (robot description, URDF)
Before this commit: robot jedy, 26 links, 25 joints
Joints:
- joint front_left_wheel_joint: limit effort=0.48 velocity=6.55 -> effort=100 velocity=6.55
- joint front_right_wheel_joint: limit effort=0.48 velocity=6.55 -> effort=100 velocity=6.55
- joint pseudo_base_joint: limit lower=0 upper=0 effort=0 velocity=0 -> (none)
- joint rear_left_wheel_joint: limit effort=0.48 velocity=6.55 -> effort=100 velocity=6.55
- joint rear_right_wheel_joint: limit effort=0.48 velocity=6.55 -> effort=100 velocity=6.55

Commit message: Add stl model

File: jedy/jedy_description/urdf/jedy.urdf (robot description, URDF)
Before this commit: robot jedy, 26 links, 25 joints
Links:
- link head_link0: geometry collision mesh filename=package://jedy_description/meshes/head_link0.stl; visual mesh filename=package://jedy_description/meshes/head_link0.dae
- link head_link1: geometry collision mesh filename=package://jedy_description/meshes/head_link1.stl; visual mesh filename=package://jedy_description/meshes/head_link1.dae
- link larm_link0: geometry collision mesh filename=package://jedy_description/meshes/larm_link0.stl; visual mesh filename=package://jedy_description/meshes/larm_link0.dae
- link larm_link1: geometry collision mesh filename=package://jedy_description/meshes/larm_link1.stl; visual mesh filename=package://jedy_description/meshes/larm_link1.dae
- link larm_link2: geometry collision mesh filename=package://jedy_description/meshes/larm_link2.stl; visual mesh filename=package://jedy_description/meshes/larm_link2.dae
- link larm_link3: geometry collision mesh filename=package://jedy_description/meshes/larm_link3.stl; visual mesh filename=package://jedy_description/meshes/larm_link3.dae
- link larm_link4: geometry collision mesh filename=package://jedy_description/meshes/larm_link4.stl; visual mesh filename=package://jedy_description/meshes/larm_link4.dae
- link larm_link5: geometry collision mesh filename=package://jedy_description/meshes/larm_link5.stl; visual mesh filename=package://jedy_description/meshes/larm_link5.dae
- link larm_link6: geometry collision mesh filename=package://jedy_description/meshes/larm_link6.stl; visual mesh filename=package://jedy_description/meshes/larm_link6.dae
- link larm_link7: geometry collision mesh filename=package://jedy_description/meshes/larm_link7.stl; visual mesh filename=package://jedy_description/meshes/larm_link7.dae
- link larm_link8: geometry collision mesh filename=package://jedy_description/meshes/larm_link8.stl; visual mesh filename=package://jedy_description/meshes/larm_link8.dae
- link rarm_link0: geometry collision mesh filename=package://jedy_description/meshes/rarm_link0.stl; visual mesh filename=package://jedy_description/meshes/rarm_link0.dae
- link rarm_link1: geometry collision mesh filename=package://jedy_description/meshes/rarm_link1.stl; visual mesh filename=package://jedy_description/meshes/rarm_link1.dae
- link rarm_link2: geometry collision mesh filename=package://jedy_description/meshes/rarm_link2.stl; visual mesh filename=package://jedy_description/meshes/rarm_link2.dae
- link rarm_link3: geometry collision mesh filename=package://jedy_description/meshes/rarm_link3.stl; visual mesh filename=package://jedy_description/meshes/rarm_link3.dae
- link rarm_link4: geometry collision mesh filename=package://jedy_description/meshes/rarm_link4.stl; visual mesh filename=package://jedy_description/meshes/rarm_link4.dae
- link rarm_link5: geometry collision mesh filename=package://jedy_description/meshes/rarm_link5.stl; visual mesh filename=package://jedy_description/meshes/rarm_link5.dae
- link rarm_link6: geometry collision mesh filename=package://jedy_description/meshes/rarm_link6.stl; visual mesh filename=package://jedy_description/meshes/rarm_link6.dae
- link rarm_link7: geometry collision mesh filename=package://jedy_description/meshes/rarm_link7.stl; visual mesh filename=package://jedy_description/meshes/rarm_link7.dae
- link rarm_link8: geometry collision mesh filename=package://jedy_description/meshes/rarm_link8.stl; visual mesh filename=package://jedy_description/meshes/rarm_link8.dae
- link real_base_link: geometry collision mesh filename=package://jedy_description/meshes/base_link.stl; visual mesh filename=package://jedy_description/meshes/base_link.dae

Commit message: Add camera link

File: jedy/jedy_description/urdf/jedy.urdf (robot description, URDF)
Before this commit: robot jedy, 26 links, 25 joints
Links:
- added link camera_depth_frame
- added link camera_depth_optical_frame
- added link camera_link, mass 0.564
Joints:
- added joint camera_depth_joint: type fixed, parent camera_link, child camera_depth_frame, origin xyz=0 0.025 0 rpy=0 0 0
- added joint camera_depth_optical_joint: type fixed, parent camera_depth_frame, child camera_depth_optical_frame, origin xyz=0 0 0 rpy=-1.5707963267948966 0 -1.5707963267948966
- added joint camera_joint: type fixed, parent head_link1, child camera_link, origin xyz=-0.031 0.0125 -0.016 rpy=0 0 0

Commit message: Add gazebo

File: jedy/jedy_description/urdf/jedy.urdf (robot description, URDF)
Before this commit: robot jedy, 29 links, 28 joints
Links:
- added link base_laser
- link front_left_wheel_link: mass 0.0620331863909222 -> 0.095024
- link front_right_wheel_link: mass 0.0620356799852319 -> 0.095024
- link head_link0: mass 0.0267722516782374 -> 0.037398
- link head_link1: mass 0.184305345878305 -> 0.093045
- link real_base_link: mass 0.642084743261537 -> 0.671312
- link rear_left_wheel_link: mass 0.0620331863909222 -> 0.095024
- link rear_right_wheel_link: mass 0.0620356799852319 -> 0.095024
Joints:
- added joint base_laser_joint: type fixed, parent base_link, child base_laser, origin xyz=0.1 0 -0.0 rpy=0 0 0

Commit message: Update vision

File: jedy/jedy_description/urdf/jedy.urdf (robot description, URDF)
Before this commit: robot jedy, 30 links, 29 joints
Links:
- added link camera_color_frame
- added link camera_color_optical_frame
Joints:
- removed joint camera_depth_joint
- removed joint camera_depth_optical_joint
- added joint camera_color_frame_joint: type fixed, parent camera_link, child camera_color_frame, origin xyz=0 0 0 rpy=0 0 0
- added joint camera_color_optical_frame_joint: type fixed, parent camera_color_frame, child camera_color_optical_frame, origin xyz=0 0 0 rpy=-1.57 0 -1.57
- added joint camera_depth_frame_joint: type fixed, parent camera_link, child camera_depth_frame, origin xyz=0 0 0 rpy=0 0 0
- added joint camera_depth_optical_frame_joint: type fixed, parent camera_depth_frame, child camera_depth_optical_frame, origin xyz=0 0 0 rpy=-1.57 0 -1.57
- joint camera_joint: origin xyz=-0.031 0.0125 -0.016 rpy=0 0 0 -> xyz=0 0.005 0.05 rpy=0 0 0

File: jedy/jedy_description/urdf/jedy_no_arm.urdf (robot description, URDF)
Before this commit: robot jedy, 12 links, 11 joints
Links:
- added link camera_color_frame
- added link camera_color_optical_frame
Joints:
- removed joint camera_depth_joint
- removed joint camera_depth_optical_joint
- added joint camera_color_frame_joint: type fixed, parent camera_link, child camera_color_frame, origin xyz=0 0 0 rpy=0 0 0
- added joint camera_color_optical_frame_joint: type fixed, parent camera_color_frame, child camera_color_optical_frame, origin xyz=0 0 0 rpy=-1.57 0 -1.57
- added joint camera_depth_frame_joint: type fixed, parent camera_link, child camera_depth_frame, origin xyz=0 0 0 rpy=0 0 0
- added joint camera_depth_optical_frame_joint: type fixed, parent camera_depth_frame, child camera_depth_optical_frame, origin xyz=0 0 0 rpy=-1.57 0 -1.57
- joint camera_joint: origin xyz=-0.031 0.0125 -0.016 rpy=0 0 0 -> xyz=0 0.005 0.05 rpy=0 0 0
