Commit message: [jedy_bringup] Publish camera from camera_color_optical_frame

File: jedy/jedy_description/urdf/jedy_gz.xacro (robot description, xacro)
@@ -690,5 +690,5 @@
     <child link="camera_link"/>
     <axis xyz="1. 0. 0."/>
-    <origin xyz="0.0 0.015 0.08" rpy="0.0 -0.0 0.0"/>
+    <origin xyz="0.02 0.01 0.06" rpy="0.0 -0.0 0.0"/>
   </joint>
   <joint name="camera_color_frame_joint" type="fixed">
@@ -962,5 +962,5 @@
       <visualize>true</visualize>
       <topic>camera</topic>
-      <frame_id>camera_depth_optical_frame</frame_id>
+      <gz_frame_id>camera_color_optical_frame</gz_frame_id>
       <camera name="camera">
         <horizontal_fov>1.0471975511965976</horizontal_fov>

Commit message: [jedy_description/jedyeus] Fixed gripper mimic direction

File: jedy/jedy_description/urdf/jedy_gz.xacro (robot description, xacro)
@@ -565,16 +565,16 @@
   </joint>
   <joint name="rarm_gripper_joint" type="revolute">
-    <limit effort="0.48" velocity="6.55" lower="-1.57" upper="0.5"/>
+    <limit effort="0.48" velocity="6.55" lower="-0.5" upper="1.57"/>
     <parent link="rarm_link6"/>
     <child link="rarm_link7"/>
-    <axis xyz="1. 0. 0."/>
+    <axis xyz="-1. 0. 0."/>
     <origin xyz="0.0 -0.011737 -0.056303" rpy="0.0 -0.0 0.0"/>
   </joint>
   <joint name="rarm_mimic_gripper_joint" type="revolute">
-    <limit effort="0.48" velocity="6.55" lower="-0.5" upper="1.57"/>
+    <limit effort="0.48" velocity="6.55" lower="-1.57" upper="0.5"/>
     <mimic joint="rarm_gripper_joint" multiplier="-1.0" offset="0.0"/>
     <parent link="rarm_link6"/>
     <child link="rarm_link8"/>
-    <axis xyz="1. 0. 0."/>
+    <axis xyz="-1. 0. 0."/>
     <origin xyz="0.0 0.011741 -0.056303" rpy="0.0 -0.0 0.0"/>
   </joint>
